File: pcb/lo_cate_pcb.kicad_sch (KiCad schematic)
At the start: 57 parts, among them J2 690-005-299-043, J3 Conn_01x09_Pin, SW1 MICRO_RESET, SW2 MICRO_ON, SW3 BUTTON1, SW4 BUTTON2, SW5 BUTTON3, U1 STM32F401RETx, U2 BMI323, U3 LED1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

Commit message: Made changes the PCB to take it to version 2, bom just needs updating now
Parts:
- removed TP1: TP_IMU_MISO, TestPoint:TestPoint_Pad_D2.0mm, symbol Connector:TestPoint
- removed TP2: TP_IMU_MOSI, TestPoint:TestPoint_Pad_D2.0mm, symbol Connector:TestPoint
- removed TP3: TP_LORA_MISO, TestPoint:TestPoint_Pad_D2.0mm, symbol Connector:TestPoint
- removed TP4: TP_LORA_MOSI, TestPoint:TestPoint_Pad_D2.0mm, symbol Connector:TestPoint
- removed U3: LED1, footprints:150141M173100_WRE-M, symbol 2024-06-21_22-48-27:150141M173100
- removed U4: LED2, footprints:150141M173100_WRE-M, symbol 2024-06-21_22-48-27:150141M173100
- removed U5: LED3, footprints:150141M173100_WRE-M, symbol 2024-06-21_22-48-27:150141M173100
- added D1, D2, D3: WL-SFTW_3528_PLCC4, footprints:WL-SFTW_3528_PLCC4, symbol WL-SFTW_3528_PLCC4:WL-SFTW_3528_PLCC4
- added J1: Conn_01x05_Pin, Connector_PinSocket_2.54mm:PinSocket_1x05_P2.54mm_Vertical, symbol Connector:Conn_01x05_Pin
- added J4: Conn_01x03_Pin, Connector_PinSocket_2.54mm:PinSocket_1x03_P2.54mm_Vertical, symbol Connector:Conn_01x03_Pin
- added R15: 4.7K, Resistor_SMD:R_0805_2012Metric_Pad1.20x1.40mm_HandSolder, symbol Device:R
- C18, C19: value 10p -> 12p
- J3: footprint Connector_PinSocket_1.27mm:PinSocket_1x09_P1.27mm_Vertical -> Connector_PinSocket_2.54mm:PinSocket_1x09_P2.54mm_Vertical
- R14: value 30R -> 4.7K
Connections:
- net 3V3: now also R14.1, D1.1, D2.1, D3.1, R15.1
- net LORA_CSB: now also J1.4 (Pin_4)
- net LORA_MISO: now also J1.1 (Pin_1)
- net LORA_MOSI: now also J1.2 (Pin_2)
- net LORA_RST: now also J1.5 (Pin_5)
- net LORA_SCK: now also J1.3 (Pin_3)
- net OSC_OUT: now also C19.1, Y1.3; no longer R14.2
- net at R2.2: now also D2.2
- net at R3.1: now also D2.3
- net at R4.1: now also D2.4
- net IMU_SDA: now reaches U1.40 (PC9)
- net IMU_SDA: now also R14.2, U2.14 (SDX), J4.2 (Pin_2)
- net IMU_SCL: now reaches U1.41 (PA8)
- net IMU_SCL: now also U2.13 (SCX), J4.3 (Pin_3), R15.2
- net IMU_SA0: now reaches U1.42 (PA9)
- net IMU_SA0: now also U2.1 (SDO), J4.1 (Pin_1)
- net LORA_DIO0: now reaches U1.51 (PC10)
- net LORA_DIO0: now also U6.14 (DIO0)
- net LORA_DIO1: now reaches U1.52 (PC11)
- net LORA_DIO1: now also U6.15 (DIO1)
- net LORA_DIO2: now reaches U1.53 (PC12)
- net LORA_DIO2: now also U6.16 (DIO2)
- net at R7.2: now also D1.2
- net IMU_INT1: now reaches U2.4 (INT1)
- net IMU_INT1: now also U1.21 (PA5)
- net IMU_INT2: now reaches U2.9 (INT2)
- net IMU_INT2: now also U1.22 (PA6)
- net at R6.1: now also D1.4
- net at R5.1: now also D1.3
- net at R8.2: now also D3.2
- net at R9.1: now also D3.3
- net at R10.1: now also D3.4
- net IMU_CSB: no longer names the net of U1.24 (PC4)
- net IMU_CSB: no longer U2.12 (CSB)
- removed net IMU_MISO: U1.22 (PA6), U2.1 (SDO)
- net IMU_MOSI: no longer names the net of U1.23 (PA7)
- net IMU_MOSI: no longer U2.14 (SDX)
- removed net IMU_SCK: U1.21 (PA5), U2.13 (SCX)
- no-connect marks 8 -> 18
Other:
- moved on the sheet: C16, C17, C18, C19, H1, H2, H3, H4, J2, J3, R10, R2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
